File: device/hardware/TMA-1.kicad_pcb (KiCad board)
At the start: 2 copper layers, 68 parts, among them J1 MAIN I/O, J2 I2C, Q1 2N3904, Q2 2N3904, Q3 2N3904, Q4 2N3904, Q5 2N3904, Q6 2N3904, Q7 2N3904, Q8 2N3904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

Commit message: update: complete PCB artwork
Parts:
- added REF**: MountingHole_3mm_Pad, MountingHole:MountingHole_3mm_Pad, F.Cu at (78.7, 35.7)
- added REF**: MountingHole_3mm_Pad, MountingHole:MountingHole_3mm_Pad, F.Cu at (210.3, 35.7)
- added REF**: MountingHole_3mm_Pad, MountingHole:MountingHole_3mm_Pad, F.Cu at (210.3, 153.0)
- added REF**: MountingHole_3mm_Pad, MountingHole:MountingHole_3mm_Pad, F.Cu at (78.7, 153.0)
- moved D1 238.8 mm to (81.0, 132.1), turned to 0 degrees
- moved D2 230.0 mm to (88.6, 132.1), turned to 0 degrees
- moved D3 221.3 mm to (96.2, 132.1), turned to 0 degrees
- moved D4 212.8 mm to (103.8, 132.1), turned to 0 degrees
- moved D5 204.6 mm to (111.4, 132.1), turned to 0 degrees
- moved D6 196.6 mm to (119.0, 132.1), turned to 0 degrees
- moved Q1 129.6 mm to (86.0, 155.4), turned to 90 degrees
- moved U7 122.0 mm to (169.3, 123.6), turned to -90 degrees
- moved Q2 121.9 mm to (92.3, 155.4), turned to 90 degrees
- moved Q3 114.4 mm to (98.7, 155.4), turned to 90 degrees
- moved J1 108.9 mm to (157.1, 47.2)
- moved U1 108.3 mm to (110.2, 82.0)
- moved Q4 107.0 mm to (105.0, 155.4), turned to 90 degrees
- moved U8 106.7 mm to (205.1, 74.9)
- moved SW1 106.6 mm to (203.0, 69.0)
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Connections:
- Q6 pad 3: /STM_DIN6 -> /STM_DIN5
- Q7 pad 3: /STM_DIN5 -> /STM_DIN6
- R16 pad 1: /DIN6 -> +3.3V
- R16 pad 2: Net-(Q6-B) -> /STM_DIN4
- R17 pad 1: +3.3V -> /DIN5
- R17 pad 2: /STM_DIN4 -> Net-(Q6-B)
- R18 pad 2: /STM_DIN6 -> /STM_DIN5
- R19 pad 1: /DIN5 -> /DIN6
- R20 pad 1: /DIN7 -> +3.3V
- R20 pad 2: Net-(Q8-B) -> /STM_DIN6
- R21 pad 1: +3.3V -> /DIN7
- R21 pad 2: /STM_DIN5 -> Net-(Q8-B)
- R7 pad 1: +3.3V -> /DIN0
- R7 pad 2: /STM_DIN0 -> Net-(Q1-B)
- R8 pad 1: /DIN0 -> +3.3V
- R8 pad 2: Net-(Q1-B) -> /STM_DIN0
Routing:
- net +3.3V: track 0.00 -> 315.8 mm
- net /ESP_I2C_SDA: track 0.00 -> 222.0 mm
- net /ESP_I2C_SCL: track 0.00 -> 216.1 mm
- net /LOG_UART_RX: track 0.00 -> 210.2 mm
- net /PIN0: track 0.00 -> 206.9 mm
- net /LOG_UART_TX: track 0.00 -> 204.6 mm
- net /DEBUG_UART_RX: track 0.00 -> 203.3 mm
- net /GPS_UART_RX: track 0.00 -> 201.3 mm
- net /PIN1: track 0.00 -> 199.0 mm
- net /GPS_UART_TX: track 0.00 -> 197.3 mm
- net /DEBUG_UART_TX: track 0.00 -> 188.2 mm
- net /PIN3: track 0.00 -> 182.1 mm
- net VBUS: track 0.00 -> 177.9 mm, vias 0 -> 2
- net /PIN2: track 0.00 -> 168.6 mm
- net /ESP_COMM: track 0.00 -> 153.9 mm
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Other:
- board outline added: 141.7 x 127.5 mm
- board text added: "ANALOG"
- board text added: "CAN"
- board text added: "DIGITAL"
- board text added: "GPS"
- board text added: "LUFT-AQUILA"
- board text added: "Monolith TMA-1 Datalogger v1.0"
- board text added: "PULSE"
- board text added: "TELEMETRY"
- board text added: "https://github.com/luftaquila/monolith"
- board text added: "https://luftaquila.io"

Commit message: add: PCB v1.0 gerber files
Parts:
- U2: value NODEMCU32S -> NodeMCU-32S
- moved R25 0.74 mm to (179.5, 59.5)
- moved R26 0.74 mm to (179.5, 72.0)
- moved R27 0.74 mm to (182.6, 59.5)
- moved R28 0.74 mm to (182.6, 72.0)
- moved R29 0.74 mm to (185.6, 59.5)
- moved R30 0.74 mm to (185.6, 72.0)
- moved R31 0.74 mm to (188.7, 59.5)
- moved R32 0.74 mm to (188.7, 72.0)
Routing:
- net /DEBUG_UART_TX: track 188.2 -> 174.9 mm
- net /DEBUG_UART_RX: track 203.3 -> 190.2 mm
- net /LOG_UART_TX: track 204.6 -> 191.8 mm
- net /LOG_UART_RX: track 210.2 -> 198.1 mm
- net /PIN0: track 206.9 -> 198.9 mm
- net /PIN1: track 199.0 -> 191.2 mm
- net /PIN3: track 182.1 -> 174.3 mm
- net /PIN2: track 168.6 -> 160.8 mm
- net /GPS_UART_RX: track 201.3 -> 199.6 mm
- net /STM_PIN3: track 130.2 -> 128.8 mm
- net /GPS_UART_TX: track 197.3 -> 196.0 mm
- net /AIN3: track 8.77 -> 9.62 mm
- net /AIN0: track 13.9 -> 14.6 mm
- net /AIN1: track 7.86 -> 8.63 mm
- net VBUS: track 177.9 -> 177.2 mm
- added copper zone on B.Cu, net GND
- added copper zone on F.Cu, net GND
Other:
- board size 141.7 x 127.5 mm -> 143.8 x 129.5 mm
