File: device/hardware/TMA-1.kicad_sch (KiCad schematic)
At the start: 68 parts, among them J1 MAIN I/O, J2 I2C, Q1 2N3904, Q2 2N3904, Q3 2N3904, Q4 2N3904, Q5 2N3904, Q6 2N3904, Q7 2N3904, Q8 2N3904, SW1 CAN_{SW}, U1 STM32F407VETx, U2 NODEMCU32S, U3 MP1584EN-3.3, U4 LM393, U5 LM393, U6 ADXL345, U7 NEO-7M, U8 SN65HVD230

Commit message: update: complete PCB artwork
Parts:
- renumbered Q7 to Q6, Q6 to Q7, R17 to R16, R19 to R17, R21 to R18, R16 to R19, R18 to R20, R20 to R21, R8 to R7, R7 to R8
Changed lines of the file:
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@@
   (symbol (lib_id "Transistor_BJT:2N3904") (at 171.45 124.46 0) (unit 1)
     (in_bom yes) (on_board yes) (dnp no) (fields_autoplaced)
-    (property "Reference" "Q7" (at 176.53 123.19 0)
+    (property "Reference" "Q6" (at 176.53 123.19 0)
       (effects (font (size 1.27 1.27)) (justify left))
     )
@@
       (project "TMA-1"
         (path "/d67581b5-2556-4cd6-beba-bc1f772a35d2"
-          (reference "Q7") (unit 1)
+          (reference "Q6") (unit 1)
         )
       )
@@
   (symbol (lib_id "Device:R_US") (at 120.65 50.8 90) (unit 1)
     (in_bom yes) (on_board yes) (dnp no)
-    (property "Reference" "R8" (at 120.65 47.625 90)
+    (property "Reference" "R7" (at 120.65 47.625 90)
       (effects (font (size 1.27 1.27)))
     )
@@
       (project "TMA-1"
         (path "/d67581b5-2556-4cd6-beba-bc1f772a35d2"
-          (reference "R8") (unit 1)
+          (reference "R7") (unit 1)
         )
       )
@@
   (symbol (lib_id "Transistor_BJT:2N3904") (at 129.54 161.29 0) (unit 1)
     (in_bom yes) (on_board yes) (dnp no) (fields_autoplaced)
-    (property "Reference" "Q6" (at 134.62 160.02 0)
+    (property "Reference" "Q7" (at 134.62 160.02 0)
       (effects (font (size 1.27 1.27)) (justify left))
     )
@@
       (project "TMA-1"
         (path "/d67581b5-2556-4cd6-beba-bc1f772a35d2"
-          (reference "Q6") (unit 1)
+          (reference "Q7") (unit 1)
         )
       )
@@
   (symbol (lib_id "Device:R_US") (at 132.08 111.76 0) (unit 1)
     (in_bom yes) (on_board yes) (dnp no) (fields_autoplaced)
-    (property "Reference" "R17" (at 133.985 110.49 0)
+    (property "Reference" "R16" (at 134.62 110.49 0)
       (effects (font (size 1.27 1.27)) (justify left))
     )
-    (property "Value" "1k" (at 133.985 113.03 0)
+    (property "Value" "1k" (at 134.62 113.03 0)
       (effects (font (size 1.27 1.27)) (justify left))
     )
@@
       (project "TMA-1"
         (path "/d67581b5-2556-4cd6-beba-bc1f772a35d2"
-          (reference "R17") (unit 1)
+          (reference "R16") (unit 1)
         )
       )
@@
   (symbol (lib_id "Device:R_US") (at 132.08 148.59 0) (unit 1)
     (in_bom yes) (on_board yes) (dnp no) (fields_autoplaced)
-    (property "Reference" "R18" (at 133.985 147.32 0)
+    (property "Reference" "R20" (at 134.62 147.32 0)
       (effects (font (size 1.27 1.27)) (justify left))
     )
-    (property "Value" "1k" (at 133.985 149.86 0)
+    (property "Value" "1k" (at 134.62 149.86 0)
       (effects (font (size 1.27 1.27)) (justify left))
     )
@@
       (project "TMA-1"
         (path "/d67581b5-2556-4cd6-beba-bc1f772a35d2"
-          (reference "R18") (unit 1)
+          (reference "R20") (unit 1)
         )
       )
@@
   (symbol (lib_id "Device:R_US") (at 132.08 38.1 0) (unit 1)
     (in_bom yes) (on_board yes) (dnp no) (fields_autoplaced)
-    (property "Reference" "R7" (at 133.985 36.83 0)
+    (property "Reference" "R8" (at 134.62 36.83 0)
       (effects (font (size 1.27 1.27)) (justify left))
     )
-    (property "Value" "1k" (at 133.985 39.37 0)
+    (property "Value" "1k" (at 134.62 39.37 0)
       (effects (font (size 1.27 1.27)) (justify left))
     )
@@
       (project "TMA-1"
         (path "/d67581b5-2556-4cd6-beba-bc1f772a35d2"
-          (reference "R7") (unit 1)
+          (reference "R8") (unit 1)
         )
       )
@@
   )
   (symbol (lib_id "Device:R_US") (at 173.99 148.59 0) (unit 1)
-    (in_bom yes) (on_board yes) (dnp no) (fields_autoplaced)
-    (property "Reference" "R22" (at 175.895 147.32 0)
+    (in_bom yes) (on_board yes) (dnp no)
+    (property "Reference" "R22" (at 176.53 147.32 0)
       (effects (font (size 1.27 1.27)) (justify left))
     )
-    (property "Value" "1k" (at 175.895 149.86 0)
+    (property "Value" "1k" (at 176.53 149.86 0)
       (effects (font (size 1.27 1.27)) (justify left))
     )
@@
   (symbol (lib_id "Device:R_US") (at 120.65 161.29 90) (unit 1)
     (in_bom yes) (on_board yes) (dnp no)
-    (property "Reference" "R16" (at 120.65 158.115 90)
+    (property "Reference" "R19" (at 120.65 158.115 90)
       (effects (font (size 1.27 1.27)))
     )
@@
       (project "TMA-1"
         (path "/d67581b5-2556-4cd6-beba-bc1f772a35d2"
-          (reference "R16") (unit 1)
+          (reference "R19") (unit 1)
         )
       )
@@
   (symbol (lib_id "Device:R_US") (at 162.56 124.46 90) (unit 1)
     (in_bom yes) (on_board yes) (dnp no)
-    (property "Reference" "R19" (at 162.56 121.285 90)
+    (property "Reference" "R17" (at 162.56 121.285 90)
       (effects (font (size 1.27 1.27)))
     )
@@
       (project "TMA-1"
         (path "/d67581b5-2556-4cd6-beba-bc1f772a35d2"
-          (reference "R19") (unit 1)
+          (reference "R17") (unit 1)
         )
       )
@@
   (symbol (lib_id "Device:R_US") (at 173.99 111.76 0) (unit 1)
     (in_bom yes) (on_board yes) (dnp no) (fields_autoplaced)
-    (property "Reference" "R21" (at 175.895 110.49 0)
+    (property "Reference" "R18" (at 176.53 110.49 0)
       (effects (font (size 1.27 1.27)) (justify left))
     )
-    (property "Value" "1k" (at 175.895 113.03 0)
+    (property "Value" "1k" (at 176.53 113.03 0)
       (effects (font (size 1.27 1.27)) (justify left))
     )
@@
       (project "TMA-1"
         (path "/d67581b5-2556-4cd6-beba-bc1f772a35d2"
-          (reference "R21") (unit 1)
+          (reference "R18") (unit 1)
         )
       )
@@
   (symbol (lib_id "Device:R_US") (at 162.56 161.29 90) (unit 1)
     (in_bom yes) (on_board yes) (dnp no)
-    (property "Reference" "R20" (at 162.56 158.115 90)
+    (property "Reference" "R21" (at 162.56 158.115 90)
       (effects (font (size 1.27 1.27)))
     )
@@
       (project "TMA-1"
         (path "/d67581b5-2556-4cd6-beba-bc1f772a35d2"
-          (reference "R20") (unit 1)
+          (reference "R21") (unit 1)
         )
       )

Commit message: improve: PCB v1.1 add debug uart jumper
Parts:
- removed J2: I2C, Connector_Molex:Molex_SPOX_5267-02A_1x02_P2.50mm_Vertical, symbol Connector_Generic:Conn_01x02
- added J2: DEBUG, Connector_PinHeader_2.54mm:PinHeader_1x03_P2.54mm_Vertical, symbol Connector_Generic:Conn_01x03
- renumbered C2 to C1
Connections:
- net DEBUG_UART_RX: now also J2.2 (Pin_2); no longer J1.22 (Pin_22)
- net DEBUG_UART_TX: now also J2.1 (Pin_1); no longer J1.10 (Pin_10)
- net ESP_I2C_SCL: now also J1.23 (Pin_23)
- net ESP_I2C_SDA: now also J1.11 (Pin_11)
- net GND: now also J2.3 (Pin_3)
- net LOG_UART_RX: now also J1.22 (Pin_22); no longer J1.23 (Pin_23)
- net LOG_UART_TX: now also J1.10 (Pin_10); no longer J1.11 (Pin_11)
Other:
- moved on the sheet: J1, R41, R42

Commit message: fix: misc bugs PCB v1.2
Parts:
- R1, R2, R3, R4, R5, R6: value 100 -> 220
Connections:
- net GND: now also U2.GND@2
- no-connect marks 99 -> 98
Other:
- moved on the sheet: R41, R42
Changed lines of the file:
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@@
 (kicad_sch (version 20230121) (generator eeschema)
   (paper "A3")
-  (junction (at 257.81 64.77) (diameter 0) (color 0 0 0 0)
-  )
   (junction (at 118.745 254) (diameter 0) (color 0 0 0 0)
   )
@@
   (junction (at 132.08 117.475) (diameter 0) (color 0 0 0 0)
   )
-  (junction (at 254.635 47.625) (diameter 0) (color 0 0 0 0)
+  (junction (at 257.81 47.625) (diameter 0) (color 0 0 0 0)
   )
   (junction (at 247.65 155.575) (diameter 0) (color 0 0 0 0)
   )
+  (junction (at 260.985 64.77) (diameter 0) (color 0 0 0 0)
+  )
   (junction (at 173.99 154.305) (diameter 0) (color 0 0 0 0)
   )
@@
   (junction (at 132.08 80.645) (diameter 0) (color 0 0 0 0)
   )
-  (junction (at 254.635 72.39) (diameter 0) (color 0 0 0 0)
-  )
   (junction (at 168.91 230.505) (diameter 0) (color 0 0 0 0)
   )
@@
   (junction (at 61.595 246.38) (diameter 0) (color 0 0 0 0)
   )
+  (junction (at 257.81 72.39) (diameter 0) (color 0 0 0 0)
+  )
   (junction (at 173.99 117.475) (diameter 0) (color 0 0 0 0)
   )
@@
   (no_connect (at 328.295 38.1))
   (no_connect (at 213.995 72.39))
-  (no_connect (at 252.095 59.69))
   (no_connect (at 338.455 38.1))
   (no_connect (at 351.155 99.06))
@@
     (stroke (width 0) (type default))
   )
-  (wire (pts (xy 252.095 64.77) (xy 257.81 64.77))
+  (wire (pts (xy 252.095 64.77) (xy 260.985 64.77))
     (stroke (width 0) (type default))
   )
@@
     (stroke (width 0) (type default))
   )
-  (wire (pts (xy 252.095 72.39) (xy 254.635 72.39))
-    (stroke (width 0) (type default))
-  )
   (wire (pts (xy 132.08 117.475) (xy 132.08 119.38))
     (stroke (width 0) (type default))
@@
     (stroke (width 0) (type default))
   )
+  (wire (pts (xy 255.27 59.69) (xy 255.27 60.96))
+    (stroke (width 0) (type default))
+  )
   (wire (pts (xy 190.5 200.025) (xy 187.325 200.025))
     (stroke (width 0) (type default))
@@
     (stroke (width 0) (type default))
   )
+  (wire (pts (xy 252.095 59.69) (xy 255.27 59.69))
+    (stroke (width 0) (type default))
+  )
   (wire (pts (xy 59.69 42.545) (xy 59.69 40.005))
     (stroke (width 0) (type default))
@@
     (stroke (width 0) (type default))
   )
-  (wire (pts (xy 257.81 57.15) (xy 257.81 64.77))
+  (wire (pts (xy 260.985 57.15) (xy 260.985 64.77))
     (stroke (width 0) (type default))
   )
@@
     (stroke (width 0) (type default))
   )
-  (wire (pts (xy 254.635 57.15) (xy 254.635 72.39))
-    (stroke (width 0) (type default))
-  )
   (wire (pts (xy 53.975 104.14) (xy 53.975 100.965))
     (stroke (width 0) (type default))
   )
-  (wire (pts (xy 254.635 47.625) (xy 254.635 49.53))
+  (wire (pts (xy 257.81 47.625) (xy 257.81 49.53))
     (stroke (width 0) (type default))
   )
@@
     (stroke (width 0) (type default))
   )
-  (wire (pts (xy 254.635 72.39) (xy 272.415 72.39))
+  (wire (pts (xy 252.095 72.39) (xy 257.81 72.39))
     (stroke (width 0) (type default))
   )
@@
     (stroke (width 0) (type default))
   )
+  (wire (pts (xy 257.81 57.15) (xy 257.81 72.39))
+    (stroke (width 0) (type default))
+  )
   (wire (pts (xy 242.57 257.175) (xy 244.475 257.175))
     (stroke (width 0) (type default))
@@
     (stroke (width 0) (type default))
   )
-  (wire (pts (xy 254.635 45.72) (xy 254.635 47.625))
+  (wire (pts (xy 257.81 45.72) (xy 257.81 47.625))
     (stroke (width 0) (type default))
   )
@@
     (stroke (width 0) (type default))
   )
-  (wire (pts (xy 257.81 64.77) (xy 272.415 64.77))
-    (stroke (width 0) (type default))
-  )
   (wire (pts (xy 230.505 204.47) (xy 233.68 204.47))
     (stroke (width 0) (type default))
@@
     (stroke (width 0) (type default))
   )
-  (wire (pts (xy 254.635 47.625) (xy 257.81 47.625))
+  (wire (pts (xy 257.81 47.625) (xy 260.985 47.625))
     (stroke (width 0) (type default))
   )
@@
     (stroke (width 0) (type default))
   )
-  (wire (pts (xy 257.81 47.625) (xy 257.81 49.53))
+  (wire (pts (xy 260.985 47.625) (xy 260.985 49.53))
     (stroke (width 0) (type default))
   )
@@
     (stroke (width 0) (type default))
   )
+  (wire (pts (xy 257.81 72.39) (xy 273.685 72.39))
+    (stroke (width 0) (type default))
+  )
   (wire (pts (xy 114.935 230.505) (xy 114.935 231.775))
     (stroke (width 0) (type default))
@@
     (stroke (width 0) (type default))
   )
+  (wire (pts (xy 260.985 64.77) (xy 273.685 64.77))
+    (stroke (width 0) (type default))
+  )
   (wire (pts (xy 76.2 200.025) (xy 73.025 200.025))
     (stroke (width 0) (type default))
@@
     (effects (font (size 1.27 1.27)) (justify left bottom))
   )
-  (label "ESP_I2C_SCL" (at 272.415 72.39 180) (fields_autoplaced)
+  (label "ESP_I2C_SCL" (at 273.685 72.39 180) (fields_autoplaced)
     (effects (font (size 1.27 1.27)) (justify right bottom))
   )
@@
     (effects (font (size 1.27 1.27)) (justify left bottom))
   )
-  (label "ESP_I2C_SDA" (at 272.415 64.77 180) (fields_autoplaced)
+  (label "ESP_I2C_SDA" (at 273.685 64.77 180) (fields_autoplaced)
     (effects (font (size 1.27 1.27)) (justify right bottom))
   )
@@
       (effects (font (size 1.27 1.27)))
     )
-    (property "Value" "100" (at 70.485 144.145 90)
+    (property "Value" "220" (at 70.485 144.145 90)
       (effects (font (size 1.27 1.27)))
     )
@@
       (effects (font (size 1.27 1.27)))
     )
-    (property "Value" "100" (at 70.485 130.81 90)
+    (property "Value" "220" (at 70.485 130.81 90)
       (effects (font (size 1.27 1.27)))
     )
@@
     )
   )
+  (symbol (lib_id "power:GND") (at 255.27 60.96 0) (mirror y) (unit 1)
+    (in_bom yes) (on_board yes) (dnp no)
+    (property "Reference" "#PWR09" (at 255.27 67.31 0)
+      (effects (font (size 1.27 1.27)) hide)
+    )
+    (property "Value" "GND" (at 255.27 58.42 0)
+      (effects (font (size 1.27 1.27)))
+    )
+    (property "Footprint" "" (at 255.27 60.96 0)
+      (effects (font (size 1.27 1.27)) hide)
+    )
+    (property "Datasheet" "" (at 255.27 60.96 0)
+      (effects (font (size 1.27 1.27)) hide)
+    )
+    (pin "1")
+    (instances
+      (project "TMA-1"
+        (path "/d67581b5-2556-4cd6-beba-bc1f772a35d2"
+          (reference "#PWR09") (unit 1)
+        )
+      )
+    )
+  )
   (symbol (lib_id "Device:LED") (at 60.325 127.635 0) (mirror x) (unit 1)
     (in_bom yes) (on_board yes) (dnp no)
@@
       (effects (font (size 1.27 1.27)))
     )
-    (property "Value" "100" (at 70.485 104.14 90)
+    (property "Value" "220" (at 70.485 104.14 90)
       (effects (font (size 1.27 1.27)))
     )
@@
     )
   )
-  (symbol (lib_id "Device:R_US") (at 257.81 53.34 0) (unit 1)
+  (symbol (lib_id "Device:R_US") (at 260.985 53.34 0) (unit 1)
     (in_bom yes) (on_board yes) (dnp no)
-    (property "Reference" "R42" (at 259.715 52.07 0)
+    (property "Reference" "R42" (at 262.89 52.07 0)
       (effects (font (size 1.27 1.27)) (justify left))
     )
-    (property "Value" "2.7k" (at 259.715 54.61 0)
+    (property "Value" "2.7k" (at 262.89 54.61 0)
       (effects (font (size 1.27 1.27)) (justify left))
     )
-    (property "Footprint" "Resistor_THT:R_Axial_DIN0207_L6.3mm_D2.5mm_P10.16mm_Horizontal" (at 258.826 53.594 90)
+    (property "Footprint" "Resistor_THT:R_Axial_DIN0207_L6.3mm_D2.5mm_P10.16mm_Horizontal" (at 262.001 53.594 90)
       (effects (font (size 1.27 1.27)) hide)
     )
-    (property "Datasheet" "~" (at 257.81 53.34 0)
+    (property "Datasheet" "~" (at 260.985 53.34 0)
       (effects (font (size 1.27 1.27)) hide)
     )
@@
       (effects (font (size 1.27 1.27)))
     )
-    (property "Value" "100" (at 70.485 170.815 90)
+    (property "Value" "220" (at 70.485 170.815 90)
       (effects (font (size 1.27 1.27)))
     )
@@
     )
   )
-  (symbol (lib_id "power:+3.3V") (at 254.635 45.72 0) (unit 1)
+  (symbol (lib_id "power:+3.3V") (at 257.81 45.72 0) (unit 1)
     (in_bom yes) (on_board yes) (dnp no)
-    (property "Reference" "#PWR064" (at 254.635 49.53 0)
+    (property "Reference" "#PWR064" (at 257.81 49.53 0)
       (effects (font (size 1.27 1.27)) hide)
     )
-    (property "Value" "+3.3V" (at 254.635 41.275 0)
+    (property "Value" "+3.3V" (at 257.81 41.275 0)
       (effects (font (size 1.27 1.27)))
     )
-    (property "Footprint" "" (at 254.635 45.72 0)
+    (property "Footprint" "" (at 257.81 45.72 0)
       (effects (font (size 1.27 1.27)) hide)
     )
-    (property "Datasheet" "" (at 254.635 45.72 0)
+    (property "Datasheet" "" (at 257.81 45.72 0)
       (effects (font (size 1.27 1.27)) hide)
     )
@@
     )
   )
-  (symbol (lib_id "Device:R_US") (at 254.635 53.34 0) (unit 1)
+  (symbol (lib_id "Device:R_US") (at 257.81 53.34 0) (unit 1)
     (in_bom yes) (on_board yes) (dnp no)
-    (property "Reference" "R41" (at 248.92 52.07 0)
+    (property "Reference" "R41" (at 252.095 52.07 0)
       (effects (font (size 1.27 1.27)) (justify left))
     )
-    (property "Value" "2.7k" (at 252.73 54.61 0)
+    (property "Value" "2.7k" (at 255.905 54.61 0)
       (effects (font (size 1.27 1.27)) (justify right))
     )
-    (property "Footprint" "Resistor_THT:R_Axial_DIN0207_L6.3mm_D2.5mm_P10.16mm_Horizontal" (at 255.651 53.594 90)
+    (property "Footprint" "Resistor_THT:R_Axial_DIN0207_L6.3mm_D2.5mm_P10.16mm_Horizontal" (at 258.826 53.594 90)
       (effects (font (size 1.27 1.27)) hide)
     )
-    (property "Datasheet" "~" (at 254.635 53.34 0)
+    (property "Datasheet" "~" (at 257.81 53.34 0)
       (effects (font (size 1.27 1.27)) hide)
     )
@@
       (effects (font (size 1.27 1.27)))
     )
-    (property "Value" "100" (at 70.485 117.475 90)
+    (property "Value" "220" (at 70.485 117.475 90)
       (effects (font (size 1.27 1.27)))
     )
@@
       (effects (font (size 1.27 1.27)))
     )
-    (property "Value" "100" (at 70.485 157.48 90)
+    (property "Value" "220" (at 70.485 157.48 90)
       (effects (font (size 1.27 1.27)))
     )
